File: zx-talker.kicad_pcb (KiCad board)
At the start: 2 copper layers, 75.9 x 66 mm, 33 parts, among them IC3 SP0256-AL2, J1 ZX_Spectrum_Connector_48K, Q1 BC548, U1 74LS00, U2 74LS32, U3 LM386

Commit message: updated with improvements
Parts:
- removed C13: 100nF, Capacitor_THT:C_Disc_D3.0mm_W1.6mm_P2.50mm
- removed R2: 100, Resistor_THT:R_Axial_DIN0207_L6.3mm_D2.5mm_P10.16mm_Horizontal
- removed R3: 330, Resistor_THT:R_Axial_DIN0207_L6.3mm_D2.5mm_P10.16mm_Horizontal
- removed the U1 at (51.5, 86.6)
- added C16: 100nF ceramic, Capacitor_THT:C_Disc_D3.0mm_W1.6mm_P2.50mm, F.Cu at (47.1, 82.2)
- added J2: WAIT, Connector_PinHeader_2.54mm:PinHeader_1x02_P2.54mm_Horizontal, F.Cu at (110.8, 97.7)
- added Q2: BC557, Package_TO_SOT_THT:TO-92_Inline, F.Cu at (66.3, 73.9)
- added U4: 74LS126, Package_DIP:DIP-14_W7.62mm, F.Cu at (52.0, 87.1)
- added Y1: 3.12Mhz, Crystal:Crystal_HC49-U_Vertical, F.Cu at (65.3, 62.9)
- C1: value 820pF (cer) -> 22pF ceramic; footprint Capacitor_THT:C_Disc_D4.3mm_W1.9mm_P5.00mm -> Capacitor_THT:C_Rect_L7.0mm_W2.5mm_P5.00mm
- C10, C15, C3, C4: value 100nF, MKT -> 100nF MKT
- C11, C12: value 100uF, lyt -> 100uF electrolytic
- C14: value 100nF -> 100nF ceramic
- C2: value 220pF (cer) -> 22pF ceramic; footprint Capacitor_THT:C_Disc_D4.3mm_W1.9mm_P5.00mm -> Capacitor_THT:C_Rect_L7.0mm_W2.5mm_P5.00mm
- C5, C7: value 4,7uF, tantal -> 4,7uF tantalum
- C6: value 470pF (cer) -> 470pF ceramic
- C8: value 10uF, lyt -> 10uF electrolytic
- C9: value 100nF,MKT -> 100nF MKT
- R1: value 4.7K -> 1K; footprint Potentiometer_THT:Potentiometer_Piher_PT-10-V10_Vertical -> Resistor_THT:R_Axial_DIN0207_L6.3mm_D2.5mm_P10.16mm_Horizontal
- U2: value 74LS32 -> 74LS27
- moved R1 18.4 mm to (62.0, 72.6), turned to 180 degrees
- moved C2 12.2 mm to (53.8, 62.9), turned to 0 degrees
- moved HT1 10.1 mm to (110.8, 88.6)
- moved C1 9.89 mm to (58.8, 58.0), turned to 180 degrees
- moved R8 6.71 mm to (110.8, 77.6)
- moved C7 6.40 mm to (111.7, 67.0), turned to -90 degrees
- moved C3 4.24 mm to (65.0, 90.9), turned to 0 degrees
- moved C4 2.27 mm to (81.7, 57.7)
- moved Q1 2.24 mm to (95.2, 58.9)
- moved C15 2.23 mm to (111.6, 57.7)
- moved C6 2.23 mm to (107.3, 57.7)
- moved U2 1.73 mm to (52.1, 104.5)
- moved C5 1.05 mm to (75.8, 63.1)
- moved R9 0.68 mm to (73.1, 104.4)
- moved C11 0.45 mm to (94.5, 90.9)
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- renumbered IC3 to U1
Connections:
- C1 pad 1: Net-(C1-Pad1) -> Net-(U1-OSC_2)
- C1 pad 2: Net-(IC3-OSC_1) -> GND
- C12 pad 1: Net-(U3-V+) -> Net-(Q2-C)
- C2 pad 1: Net-(C2-Pad1) -> GND
- C2 pad 2: Net-(C2-Pad2) -> Net-(U1-OSC_1)
- J1 pad A21: unconnected-(J1-A7-PadA21) -> A7
- J1 pad A23: A5 -> unconnected-(J1-A5-PadA23)
- J1 pad B18: unconnected-(J1-RD-PadB18) -> RD
- J1 pad B3: unconnected-(J1-D7-PadB3) -> D7
- J1 pad B9: unconnected-(J1-D6-PadB9) -> D6
- R1 pad 1: Net-(IC3-OSC_1) -> Net-(Q2-B)
- R1 pad 2: Net-(R1-Pad2) -> SBY
- R10 pad 1: Net-(U3-V+) -> Net-(Q2-E)
- U1 pad 10: unconnected-(IC3-A8-Pad10) -> GND
- U1 pad 11: unconnected-(IC3-A7-Pad11) -> GND
- U1 pad 22: unconnected-(IC3-TEST-Pad22) -> GND
- U1 pad 27: Net-(IC3-OSC_1) -> Net-(U1-OSC_1)
- U1 pad 28: unconnected-(IC3-OSC_2-Pad28) -> Net-(U1-OSC_2)
- U1 pad 8: WAIT -> SBY
- U1 pad 9: unconnected-(IC3-~{LRQ}-Pad9) -> ~{LRQ}
- U2 pad 1: A5 -> WR
- U2 pad 10: GND -> IORQ
- U2 pad 11: unconnected-(U2-Pad11) -> A7
- U2 pad 12: GND -> Net-(U2-Pad12)
- U2 pad 13: GND -> A7
- U2 pad 3: Net-(U2-Pad3) -> Net-(U2-Pad12)
- U2 pad 4: Net-(U2-Pad3) -> Net-(U2-Pad12)
- U2 pad 5: WR -> Net-(U2-Pad12)
- U2 pad 8: unconnected-(U2-Pad8) -> Net-(U2-Pad8)
- U2 pad 9: GND -> RD
- U3 pad 6: Net-(U3-V+) -> Net-(Q2-C)
Routing:
- net SBY: track 0.00 -> 78.1 mm, vias 0 -> 1
- net A7: track 0.00 -> 64.7 mm, vias 0 -> 2
- net A5: track 62.3 -> 0.00 mm, vias 1 -> 0
- net GND: track 230.8 -> 287.7 mm
- net Net-(Q2-C): track 0.00 -> 47.1 mm, vias 0 -> 2
- net D7: track 0.00 -> 43.7 mm, vias 0 -> 1
- net Net-(IC3-OSC_1): track 42.5 -> 0.00 mm
- net RD: track 0.00 -> 41.4 mm, vias 0 -> 1
- net ~{LRQ}: track 0.00 -> 37.2 mm
- net D6: track 0.00 -> 31.1 mm, vias 0 -> 1
- net Net-(Q2-E): track 0.00 -> 29.6 mm
- net Net-(U2-Pad8): track 0.00 -> 27.3 mm, vias 0 -> 1
- net Net-(C1-Pad1): track 25.3 -> 0.00 mm
- net Net-(C2-Pad2): track 24.1 -> 0.00 mm
- net Net-(C2-Pad1): track 20.4 -> 0.00 mm
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Other:
- board text added: "Speaker"
- board text added: "Volume"
- board text added: "WAIT"
- board text added: "recreated in 2025 v1.1"
- board text removed: "recreated in 2025 v1.0"
