File: zx-talker.kicad_sch (KiCad schematic)
At the start: 32 parts, among them IC3 SP0256-AL2, J1 ZX_Spectrum_Connector_48K, Q1 BC548, U1 74LS00, U2 74LS32, U3 LM386

Commit message: updated with improvements
Parts:
- removed C13: 100nF, Capacitor_THT:C_Disc_D3.0mm_W1.6mm_P2.50mm, symbol Device:C
- removed R1: 4.7K, Potentiometer_THT:Potentiometer_Piher_PT-10-V10_Vertical, symbol Device:R_Trim
- removed R2: 100, Resistor_THT:R_Axial_DIN0207_L6.3mm_D2.5mm_P10.16mm_Horizontal, symbol Device:R
- removed R3: 330, Resistor_THT:R_Axial_DIN0207_L6.3mm_D2.5mm_P10.16mm_Horizontal, symbol Device:R
- removed U1: 74LS00, Package_DIP:DIP-14_W7.62mm, symbol 74xx:74LS00
- removed U2: 74LS32, Package_DIP:DIP-14_W7.62mm, symbol 74xx:74LS32
- added C16: 100nF ceramic, Capacitor_THT:C_Disc_D3.0mm_W1.6mm_P2.50mm, symbol Device:C
- added J2: WAIT, Connector_PinHeader_2.54mm:PinHeader_1x02_P2.54mm_Horizontal, symbol Connector:Conn_01x02_Pin
- added Q2: BC557, Package_TO_SOT_THT:TO-92_Inline, symbol Transistor_BJT:BC557
- added R1: 1K, Resistor_THT:R_Axial_DIN0207_L6.3mm_D2.5mm_P10.16mm_Horizontal, symbol Device:R
- added U2: 74LS27, Package_DIP:DIP-14_W7.62mm, symbol 74xx:74LS27
- added U4: 74LS126, Package_DIP:DIP-14_W7.62mm, symbol 74xx:74LS126
- added Y1: 3.12Mhz, Crystal:Crystal_HC49-U_Vertical, symbol Device:Crystal
- C1: value 820pF (cer) -> 22pF ceramic; footprint Capacitor_THT:C_Disc_D4.3mm_W1.9mm_P5.00mm -> Capacitor_THT:C_Rect_L7.0mm_W2.5mm_P5.00mm
- C10, C15, C3, C4, C9: value 100nF, MKT -> 100nF MKT
- C11, C12: value 100uF, lyt -> 100uF electrolytic
- C14: value 100nF -> 100nF ceramic
- C2: value 220pF (cer) -> 22pF ceramic; footprint Capacitor_THT:C_Disc_D4.3mm_W1.9mm_P5.00mm -> Capacitor_THT:C_Rect_L7.0mm_W2.5mm_P5.00mm
- C5, C7: value 4,7uF, tantal -> 4,7uF tantalum
- C6: value 470pF (cer) -> 470pF ceramic
- C8: value 10uF, lyt -> 10uF electrolytic
- renumbered IC3 to U1
Connections:
- net +5V: now also C16.1, U2.14 (VCC), U4.14 (VCC)
- net GND: now also C1.2, C2.1, U1.10 (A8), U1.11 (A7), U1.22 (TEST), C16.2, U2.7 (GND), U4.1, U4.10, U4.2, U4.7 (GND), U4.9
- net IORQ: now also U2.10, U2.2
- net WAIT: now also J2.1 (Pin_1); no longer U1.8 (SBY)
- net WR: now also U2.1
- net at C12.1, U3.6 (V+): now also Q2.1 (C); no longer R10.1
- net at U1.20 (~{ALD}): now also U2.6
- net at U1.27 (OSC_1): now also C2.2, Y1.1; no longer C1.2
- net at U1.28 (OSC_2): now also C1.1, Y1.2
- net ~{LRQ}: now reaches U1.9 (~{LRQ})
- net ~{LRQ}: now also U4.12
- net A7: now reaches J1.A21 (A7)
- net A7: now also U2.11, U2.13
- net RD: now reaches J1.B18 (RD)
- net RD: now also U2.9
- net D7: now reaches J1.B3 (D7)
- net D7: now also U4.11
- net D6: now reaches J1.B9 (D6)
- net D6: now also U4.6
- net A5: no longer names the net of J1.A23 (A5)
- new net: Q2.3 (E), R10.1
- new net: Q2.2 (B), R1.1
- new net: U2.8, U4.13, U4.4
- new net: U2.12, U2.3, U2.4, U2.5
- new net SBY: J2.2 (Pin_2), R1.2, U1.8 (SBY), U4.5
- no-connect marks 56 -> 46
Other:
- note added: "Address decoding"
- note added: "Amplifier"
- note added: "Clock"
- note added: "Filter"
- note added: "version 1.1 - A7, A8, TEST to GND - Clock using Crystal (as per datasheet) - Disable AMP when IC is inactive - A7 used as adressing (A7 low, 127:dk'tronics, 31:ORG, 7:Sweet Talker) - Enable SBY & LRQ output - Cleaup version 1.0 Initial version as shown in Magazine"
- moved on the sheet: C10, C11, C12, C14, C15, C3, C4, C5, C6, C7, C8, C9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
